File: pcbs/devkit/devkit.kicad_pcb (KiCad board)
At the start: 2 copper layers, 86 x 112 mm, 49 parts, among them J3 gpio_breakout, Q1 NPN, Q10 NPN, Q11 NPN, Q12 NPN, Q2 NPN, Q3 NPN, Q4 NPN, Q5 NPN, Q6 NPN, Q7 NPN, Q8 NPN, Q9 NPN, SW1 RotaryEncoder_Switch, SW2 RotaryEncoder_Switch, SW3 RotaryEncoder_Switch, SW4 SW_Push, SW5 SW_Push, SW6 SW_Push, SW7 SW_Push, U1 MCP23017_SP

Commit message: Order baseboard and devkit
Parts:
- removed Q1, Q10, Q11, Q12, Q2, Q3, Q4, Q5, Q6, Q7, Q8, Q9: NPN, Package_TO_SOT_THT:TO-92L_Inline
- D1, D2, D3, D4, D5, D6: value LED_ARGB -> LED_BGKR
- moved R13 12.5 mm to (211.5, 33.7), turned to -90 degrees
- moved R14 10.2 mm to (206.5, 33.7), turned to -90 degrees
- moved VID1 7.69 mm to (186.8, 130.0), turned to -90 degrees
- moved D1 7.50 mm to (158.0, 49.0)
- moved D2 7.50 mm to (183.0, 49.0)
- moved D3 7.50 mm to (208.0, 49.0)
- moved D4 7.50 mm to (158.0, 72.9)
- moved D5 7.50 mm to (183.0, 73.0)
- moved D6 7.50 mm to (208.0, 73.0)
- moved RV1 7.50 mm to (155.5, 64.0)
- moved RV2 7.50 mm to (180.5, 64.0)
- moved RV3 7.50 mm to (205.5, 64.0)
- moved SW1 7.50 mm to (160.5, 75.9)
- moved SW2 7.50 mm to (185.5, 75.9)
- moved SW3 7.50 mm to (210.5, 75.9)
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Connections:
- D1 pad 1: +3V3 -> unconnected-(D1-BA-Pad1)
- D1 pad 2: Net-(D1-RK) -> Net-(D1-GA)
- D1 pad 3: Net-(D1-GK) -> GND
- D1 pad 4: unconnected-(D1-BK-Pad4) -> Net-(D1-RA)
- D2 pad 1: +3V3 -> unconnected-(D2-BA-Pad1)
- D2 pad 3: Net-(D2-GK) -> GND
- D2 pad 4: unconnected-(D2-BK-Pad4) -> Net-(D2-RA)
- D3 pad 1: +3V3 -> unconnected-(D3-BA-Pad1)
- D3 pad 3: Net-(D3-GK) -> GND
- D3 pad 4: unconnected-(D3-BK-Pad4) -> Net-(D3-RA)
- D4 pad 1: +3V3 -> unconnected-(D4-BA-Pad1)
- D4 pad 3: Net-(D4-GK) -> GND
- D4 pad 4: unconnected-(D4-BK-Pad4) -> Net-(D4-RA)
- D5 pad 1: +3V3 -> unconnected-(D5-BA-Pad1)
- D5 pad 3: Net-(D5-GK) -> GND
- D5 pad 4: unconnected-(D5-BK-Pad4) -> Net-(D5-RA)
- D6 pad 1: +3V3 -> unconnected-(D6-BA-Pad1)
- D6 pad 3: Net-(D6-GK) -> GND
- D6 pad 4: unconnected-(D6-BK-Pad4) -> Net-(D6-RA)
- R1 pad 1: Net-(D1-GK) -> Net-(D1-GA)
- R1 pad 2: Net-(Q1-C) -> /LED_G_POT1
- R10 pad 2: Net-(Q10-C) -> /LED_G_ENC2
- R11 pad 1: Net-(D6-GK) -> Net-(D6-RA)
- R11 pad 2: Net-(Q11-C) -> /LED_R_ENC3
- R12 pad 2: Net-(Q12-C) -> /LED_G_ENC3
- R2 pad 1: Net-(D1-RK) -> Net-(D1-RA)
- R2 pad 2: Net-(Q2-C) -> /LED_R_POT1
- R3 pad 1: Net-(D2-GK) -> Net-(D2-RA)
- R3 pad 2: Net-(Q3-C) -> /LED_R_POT2
- R4 pad 2: Net-(Q4-C) -> /LED_G_POT2
- R5 pad 1: Net-(D3-GK) -> Net-(D3-RA)
- R5 pad 2: Net-(Q5-C) -> /LED_R_POT3
- R6 pad 2: Net-(Q6-C) -> /LED_G_POT3
- R7 pad 1: Net-(D4-GK) -> Net-(D4-RA)
- R7 pad 2: Net-(Q7-C) -> /LED_R_ENC1
- R8 pad 2: Net-(Q8-C) -> /LED_G_ENC1
- R9 pad 1: Net-(D5-GK) -> Net-(D5-RA)
- R9 pad 2: Net-(Q9-C) -> /LED_R_ENC2
Routing:
- net Net-(D4-RA): track 0.00 -> 79.3 mm, vias 0 -> 1
- net Net-(D4-GK): track 64.9 -> 0.00 mm, vias 1 -> 0
- net Net-(D5-GK): track 56.8 -> 0.00 mm, vias 1 -> 0
- net /GPIO1: track 157.0 -> 208.8 mm
- net /GPIO0: track 152.0 -> 203.3 mm, vias 1 -> 0
- net Net-(D3-RA): track 0.00 -> 49.1 mm, vias 0 -> 1
- net +3V3: track 184.3 -> 136.4 mm
- net Net-(D5-RA): track 0.00 -> 45.5 mm
- net Net-(D3-GK): track 45.1 -> 0.00 mm, vias 1 -> 0
- net Net-(D6-GK): track 43.6 -> 0.00 mm
- net Net-(D6-RA): track 0.00 -> 41.1 mm
- net Net-(D2-RA): track 0.00 -> 32.6 mm, vias 0 -> 2
- net Net-(D2-GK): track 28.2 -> 0.00 mm
- net Net-(D1-GA): track 0.00 -> 21.3 mm, vias 0 -> 1
- net Net-(D1-GK): track 21.2 -> 0.00 mm
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Other:
- outline, holes or cut-outs redrawn
- board text added: "multi-effects-pico devkit v0.1"
