File: pcbs/devkit/devkit.kicad_sch (KiCad schematic)
At the start: 49 parts, among them J3 gpio_breakout, Q1 NPN, Q10 NPN, Q11 NPN, Q12 NPN, Q2 NPN, Q3 NPN, Q4 NPN, Q5 NPN, Q6 NPN, Q7 NPN, Q8 NPN, Q9 NPN, SW1 RotaryEncoder_Switch, SW2 RotaryEncoder_Switch, SW3 RotaryEncoder_Switch, SW4 SW_Push, SW5 SW_Push, SW6 SW_Push, SW7 SW_Push, U1 MCP23017_SP

Commit message: Order baseboard and devkit
Parts:
- removed D1, D2, D3, D4, D5, D6: LED_ARGB, LED_THT:LED_D5.0mm-4_RGB, symbol Device:LED_ARGB
- removed Q1, Q10, Q11, Q12, Q2, Q3, Q4, Q5, Q6, Q7, Q8, Q9: NPN, Package_TO_SOT_THT:TO-92L_Inline, symbol Simulation_SPICE:NPN
- added D1, D2, D3, D4, D5, D6: LED_BGKR, LED_THT:LED_D5.0mm-4_RGB, symbol Device:LED_BGKR
Connections:
- net GND: now also D1.3 (K), D2.3 (K), D3.3 (K), D4.3 (K), D5.3 (K), D6.3 (K)
- net LED_G_ENC1: now also R8.2
- net LED_G_ENC2: now also R10.2
- net LED_G_ENC3: now also R12.2
- net LED_G_POT1: now also R1.2
- net LED_G_POT2: now also R4.2
- net LED_G_POT3: now also R6.2
- net LED_R_ENC1: now also R7.2
- net LED_R_ENC2: now also R9.2
- net LED_R_ENC3: now also R11.2
- net LED_R_POT1: now also R2.2
- net LED_R_POT2: now also R3.2
- net LED_R_POT3: now also R5.2
- net at R8.1: now also D4.2 (GA)
- net at R6.1: now also D3.2 (GA)
- net at R5.1: now also D3.4 (RA)
- net at R4.1: now also D2.2 (GA)
- net at R3.1: now also D2.4 (RA)
- net at R10.1: now also D5.2 (GA)
- net at R9.1: now also D5.4 (RA)
- net at R2.1: now also D1.4 (RA)
- net at R1.1: now also D1.2 (GA)
- net at R12.1: now also D6.2 (GA)
- net at R11.1: now also D6.4 (RA)
- net at R7.1: now also D4.4 (RA)
Other:
- note added: "TODO: x 10K pullups on I2C bus x Figure out which RGB leds I have (common cathode / anode? order?) x take dimensions of Jacks into account, they might be too high x figure out ergonomic ish layout and a good place for the compnoents x check fit on display x check encoder footprints x check pot stock / add to cart"
- note removed: "TODO: x 10K pullups on I2C bus - Figure out which RGB leds I have (common cathode / anode? order?) x take dimensions of Jacks into account, they might be too high x figure out ergonomic ish layout and a good place for the compnoents - check fit on display"
- moved on the sheet: R1, R2
